File: Hardware/knob_LCD/knob_LCD.kicad_sch (KiCad schematic)
At the start: 9 parts, among them J2 Conn_01x14_Socket, J2 ST77903, Q2 AO3400A

Commit message: CH224K & ST77903 symbol fix
Connections:
- net TP_SCL: now also J2.19 (TP_SCL); no longer J2.18 (TP_SCL)
- net TP_SDA: now also J2.20 (TP_SDA); no longer J2.19 (TP_SDA)
Changed lines of the file:
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@@
-(kicad_sch (version 20230221) (generator eeschema)
+(kicad_sch (version 20230409) (generator eeschema)
   (paper "A4")
   (junction (at 104.775 95.25) (diameter 0) (color 0 0 0 0)
@@
     (pin "17")
     (pin "18")
-    (pin "18")
     (pin "19")
     (pin "2")
+    (pin "20")
     (pin "21")
     (pin "22")
