File: Hardware/knob_motherboard/BLDC.kicad_sch (KiCad schematic)
At the start: 12 parts, among them M1 BLDC, U2 PDRV8311HRRWR, U3 MT6701

Commit message: drv8311 spi bugfix & ch224k CFG1 bugfix
Connections:
- net nFAULT: no longer names the net of R6.1, U2.1 (FAULT_N)
Changed lines of the file:
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@@
   (junction (at 45.085 43.18) (diameter 0) (color 0 0 0 0)
-  )
-  (junction (at 113.665 91.44) (diameter 0) (color 0 0 0 0)
   )
   (junction (at 34.925 40.64) (diameter 0) (color 0 0 0 0)
@@
     (stroke (width 0) (type default))
   )
-  (wire (pts (xy 113.665 96.52) (xy 113.665 91.44))
-    (stroke (width 0) (type default))
-  )
   (wire (pts (xy 92.075 146.685) (xy 92.075 151.765))
     (stroke (width 0) (type default))
   )
-  (wire (pts (xy 113.665 91.44) (xy 114.3 91.44))
-    (stroke (width 0) (type default))
-  )
   (wire (pts (xy 60.96 43.18) (xy 60.96 49.53))
     (stroke (width 0) (type default))
@@
     (stroke (width 0) (type default))
   )
-  (wire (pts (xy 111.76 96.52) (xy 113.665 96.52))
-    (stroke (width 0) (type default))
-  )
   (wire (pts (xy 92.075 164.465) (xy 102.235 164.465))
     (stroke (width 0) (type default))
@@
     (stroke (width 0) (type default))
   )
-  (wire (pts (xy 113.03 91.44) (xy 113.665 91.44))
+  (wire (pts (xy 113.03 91.44) (xy 114.3 91.44))
     (stroke (width 0) (type default))
   )
@@
     (effects (font (size 1.27 1.27)) (justify left))
   )
-  (hierarchical_label "nFAULT" (shape output) (at 111.76 96.52 180) (fields_autoplaced)
-    (effects (font (size 1.27 1.27)) (justify right))
-  )
   (hierarchical_label "DRV_CS" (shape input) (at 114.3 68.58 180) (fields_autoplaced)
